File: USB_C_Twitch/USB_C_Twitch.kicad_sch (KiCad schematic)
At the start: 68 parts, among them J1 Conn_01x06_Pin, J2 Conn_01x06_Pin, Q1 Q_PNP_BEC, Q2 Q_PNP_BEC, Q3 Q_PNP_BEC, Q4 Q_PMOS_GSD, Q5 Q_PMOS_GSD, Q6 Q_PNP_BEC, Q7 Q_PNP_BEC, Q8 Q_PMOS_GSD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

Commit message: add nev versions. (usb c and displayport working)
Parts:
- R13, R14, R3, R4, R5, R6: value 10K -> 40K
Connections:
- net A_SSRX+: now also U1.6 (SSBX); no longer U1.2 (SSAX)
- net A_SSRX-: now also U1.7 (SSBY); no longer U1.3 (SSAY)
- net A_SSTX+: now also U1.2 (SSAX); no longer U1.6 (SSBX)
- net A_SSTX-: now also U1.3 (SSAY); no longer U1.7 (SSBY)
- net B_SSRX+: now also U2.6 (SSBX); no longer U2.2 (SSAX)
- net B_SSRX-: now also U2.7 (SSBY); no longer U2.3 (SSAY)
- net B_SSTX+: now also U2.2 (SSAX); no longer U2.6 (SSBX)
- net B_SSTX-: now also U2.3 (SSAY); no longer U2.7 (SSBY)
- net C_SSRX+: now also U3.6 (SSBX); no longer U3.2 (SSAX)
- net C_SSRX-: now also U3.7 (SSBY); no longer U3.3 (SSAY)
- net C_SSTX+: now also U3.2 (SSAX); no longer U3.6 (SSBX)
- net C_SSTX-: now also U3.3 (SSAY); no longer U3.7 (SSBY)
Changed lines of the file:
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@@
 	)
 	(label "A_SSRX+"
-		(at 119.38 116.84 180)
+		(at 119.38 106.68 180)
 		(effects
 			(font
@@
 	)
 	(label "B_SSRX-"
-		(at 119.38 149.86 180)
+		(at 119.38 139.7 180)
 		(effects
 			(font
@@
 	)
 	(label "C_SSTX+"
-		(at 119.38 177.8 180)
+		(at 119.38 187.96 180)
 		(effects
 			(font
@@
 	)
 	(label "C_SSTX-"
-		(at 119.38 175.26 180)
+		(at 119.38 185.42 180)
 		(effects
 			(font
@@
 	)
 	(label "A_SSTX+"
-		(at 119.38 106.68 180)
+		(at 119.38 116.84 180)
 		(effects
 			(font
@@
 	)
 	(label "B_SSTX+"
-		(at 119.38 142.24 180)
+		(at 119.38 152.4 180)
 		(effects
 			(font
@@
 	)
 	(label "A_SSRX-"
-		(at 119.38 114.3 180)
+		(at 119.38 104.14 180)
 		(effects
 			(font
@@
 	)
 	(label "B_SSTX-"
-		(at 119.38 139.7 180)
+		(at 119.38 149.86 180)
 		(effects
 			(font
@@
 	)
 	(label "C_SSRX-"
-		(at 119.38 185.42 180)
+		(at 119.38 175.26 180)
 		(effects
 			(font
@@
 	)
 	(label "C_SSRX+"
-		(at 119.38 187.96 180)
+		(at 119.38 177.8 180)
 		(effects
 			(font
@@
 	)
 	(label "B_SSRX+"
-		(at 119.38 152.4 180)
+		(at 119.38 142.24 180)
 		(effects
 			(font
@@
 	)
 	(label "A_SSTX-"
-		(at 119.38 104.14 180)
+		(at 119.38 114.3 180)
 		(effects
 			(font
@@
 			)
 		)
-		(property "Value" "10K"
+		(property "Value" "40K"
 			(at 91.44 61.214 0)
 			(effects
@@
 			)
 		)
-		(property "Value" "10K"
+		(property "Value" "40K"
 			(at 83.82 61.214 0)
 			(effects
@@
 			)
 		)
-		(property "Value" "10K"
+		(property "Value" "40K"
 			(at 91.44 80.264 0)
 			(effects
@@
 			)
 		)
-		(property "Value" "10K"
+		(property "Value" "40K"
 			(at 91.44 40.894 0)
 			(effects
@@
 			)
 		)
-		(property "Value" "10K"
+		(property "Value" "40K"
 			(at 83.82 80.264 0)
 			(effects
@@
 			)
 		)
-		(property "Value" "10K"
+		(property "Value" "40K"
 			(at 83.82 40.894 0)
 			(effects
