File: USB_PD_Twitch/USB_PD_Twitch.kicad_pcb (KiCad board)
At the start: 4 copper layers, 60 x 60 mm, 96 parts, among them J3 USB3_A, J4 USB3_A, J5 USB3_A, Q3 Q_PMOS_GSD, Q4 Q_PMOS_GSD, Q5 Q_PMOS_GSD, U1 NDP1360KC, U10 CH482D, U11 CH482D, U12 CXP0650-220M-AG(22UH), U13 CXP0650-220M-AG(22UH), U14 CXP0650-220M-AG(22UH), U15 LM317L_SOT-89, U2 NDP1360KC, U3 XPD738B20, U4 NDP1360KC, U5 XPD738B20, U6 NDP1360KC, U7 XPD738B20, U8 CXP0650-220M-AG(22UH), U9 CH482D

Commit message: add nev versions. (usb c and displayport working)
Parts:
- removed the C20 at (145.1, 96.3)
- removed the R19 at (153.8, 66.8)
- removed the R38 at (146.8, 93.6)
- added C10: 100n, Capacitor_SMD:C_0603_1608Metric, F.Cu at (76.9, 54.1)
- added C11: 100u, Capacitor_SMD:CP_Elec_8x10, F.Cu at (69.1, 55.3)
- added C12: 100u, Capacitor_SMD:CP_Elec_8x10, F.Cu at (69.1, 65.1)
- added C13: 100n, Capacitor_SMD:C_0603_1608Metric, F.Cu at (76.9, 56.6)
- added C15: 100n, Capacitor_SMD:C_0603_1608Metric, F.Cu at (76.9, 61.6)
- added C16: 100n, Capacitor_SMD:C_0603_1608Metric, F.Cu at (76.9, 64.2)
- added C17: 100n, Capacitor_SMD:C_0603_1608Metric, F.Cu at (76.9, 66.7)
- added C23: 100n, Capacitor_SMD:C_0603_1608Metric, F.Cu at (97.7, 81.1)
- added C24: 100n, Capacitor_SMD:C_0603_1608Metric, F.Cu at (97.7, 83.6)
- added C25: 100n, Capacitor_SMD:C_0603_1608Metric, F.Cu at (97.7, 86.1)
- added C26: 100n, Capacitor_SMD:C_0603_1608Metric, F.Cu at (97.7, 88.6)
- added C27: 100n, Capacitor_SMD:C_0603_1608Metric, F.Cu at (97.7, 91.1)
- added C28: 22u, easyeda2kicad:C1812, F.Cu at (82.7, 102.5)
- added C29: 100n, Capacitor_SMD:C_0603_1608Metric, F.Cu at (76.9, 81.1)
- added C30: 100n, Capacitor_SMD:C_0603_1608Metric, F.Cu at (76.9, 83.6)
- added C31: 100u, Capacitor_SMD:CP_Elec_8x10, F.Cu at (69.1, 84.7)
- added C32: 100u, Capacitor_SMD:CP_Elec_8x10, F.Cu at (69.1, 94.6)
- added C33: 100n, Capacitor_SMD:C_0603_1608Metric, F.Cu at (76.9, 86.1)
- added C34: 100n, Capacitor_SMD:C_0603_1608Metric, F.Cu at (76.9, 88.6)
- added C35: 100n, Capacitor_SMD:C_0603_1608Metric, F.Cu at (76.9, 91.1)
- added C36: 100n, Capacitor_SMD:C_0603_1608Metric, F.Cu at (76.9, 93.6)
- added C37: 100n, Capacitor_SMD:C_0603_1608Metric, F.Cu at (76.9, 96.1)
- added C9: 100n, Capacitor_SMD:C_0603_1608Metric, F.Cu at (76.9, 51.6)
- added D1: LED, LED_SMD:LED_0603_1608Metric, F.Cu at (94.9, 97.0)
- added D2: LED, LED_SMD:LED_0603_1608Metric, F.Cu at (94.9, 99.6)
- added D3: LED, LED_SMD:LED_0603_1608Metric, F.Cu at (94.9, 102.2)
- added Q1: FS8205A_C908265, easyeda2kicad:SOT-23-6_L2.9-W1.6-P0.95-LS2.8-BR, F.Cu at (87.1, 57.9)
- added Q2: FS8205A_C908265, easyeda2kicad:SOT-23-6_L2.9-W1.6-P0.95-LS2.8-BR, F.Cu at (102.1, 90.7)
- added Q3: FS8205A_C908265, easyeda2kicad:SOT-23-6_L2.9-W1.6-P0.95-LS2.8-BR, F.Cu at (87.1, 87.4)
- added R1: 10K, Resistor_SMD:R_0402_1005Metric, F.Cu at (98.3, 96.7)
- added R2: 10K, Resistor_SMD:R_0402_1005Metric, F.Cu at (98.3, 98.7)
- added R23: 25K, Resistor_SMD:R_0402_1005Metric, F.Cu at (80.3, 55.3)
- added R24: 29K, Resistor_SMD:R_0402_1005Metric, F.Cu at (80.3, 57.3)
- added R25: 22R, Resistor_SMD:R_0402_1005Metric, F.Cu at (80.3, 59.3)
- added R26: 18K, Resistor_SMD:R_0402_1005Metric, F.Cu at (80.3, 61.3)
- added R27: 10m, Resistor_SMD:R_1206_3216Metric, F.Cu at (87.9, 63.9)
- added R3: 10K, Resistor_SMD:R_0402_1005Metric, F.Cu at (98.3, 100.7)
- added R30: 6m, Resistor_SMD:R_1206_3216Metric, F.Cu at (87.9, 67.3)
- added R32: 100R, Resistor_SMD:R_0402_1005Metric, F.Cu at (83.3, 57.3)
- added R33: 100K, Resistor_SMD:R_0402_1005Metric, F.Cu at (83.3, 59.3)
- added R37: 29K, Resistor_SMD:R_0402_1005Metric, F.Cu at (94.3, 80.8)
- added R41: 10K, Resistor_SMD:R_0402_1005Metric, F.Cu at (94.3, 84.8)
- added R43: 6m, Resistor_SMD:R_1206_3216Metric, F.Cu at (102.5, 86.9)
- added R44: 100K, Resistor_SMD:R_0402_1005Metric, F.Cu at (94.3, 88.8)
- added R45: 100R, Resistor_SMD:R_0402_1005Metric, F.Cu at (94.3, 90.7)
- added R46: 100K, Resistor_SMD:R_0402_1005Metric, F.Cu at (94.3, 92.7)
- added R47: 100K, Resistor_SMD:R_0402_1005Metric, F.Cu at (80.3, 80.8)
- added R48: 8K, Resistor_SMD:R_0402_1005Metric, F.Cu at (80.3, 82.8)
- added R49: 25K, Resistor_SMD:R_0402_1005Metric, F.Cu at (80.3, 84.8)
- added R50: 29K, Resistor_SMD:R_0402_1005Metric, F.Cu at (80.3, 86.8)
- added R51: 22R, Resistor_SMD:R_0402_1005Metric, F.Cu at (80.3, 88.8)
- added R52: 18K, Resistor_SMD:R_0402_1005Metric, F.Cu at (80.3, 90.7)
- added R53: 10m, Resistor_SMD:R_1206_3216Metric, F.Cu at (87.9, 93.4)
- added R54: 10K, Resistor_SMD:R_0402_1005Metric, F.Cu at (83.3, 80.8)
- added R55: 10K, Resistor_SMD:R_0402_1005Metric, F.Cu at (83.3, 82.8)
- added R56: 6m, Resistor_SMD:R_1206_3216Metric, F.Cu at (87.9, 96.7)
- added R57: 100K, Resistor_SMD:R_0402_1005Metric, F.Cu at (83.3, 84.8)
- added R58: 100R, Resistor_SMD:R_0402_1005Metric, F.Cu at (83.3, 86.8)
- added R59: 100K, Resistor_SMD:R_0402_1005Metric, F.Cu at (83.3, 88.8)
- added U12: TPS25740ARGER, easyeda2kicad:VQFN-24_L4.0-W4.0-P0.50-TL-EP, F.Cu at (103.2, 82.5)
- added U13: NDP1360KC, easyeda2kicad:SOP-8_L4.9-W3.9-P1.27-LS6.0-BL, F.Cu at (82.0, 95.8)
- added U14: CXP0650-220M-AG(22UH), easyeda2kicad:IND-SMD_L7.1-W6.6_CXP0650, F.Cu at (67.8, 103.4)
- added U15: TPS25740ARGER, easyeda2kicad:VQFN-24_L4.0-W4.0-P0.50-TL-EP, F.Cu at (88.1, 82.5)
- added U7: NDP1360KC, easyeda2kicad:SOP-8_L4.9-W3.9-P1.27-LS6.0-BL, F.Cu at (82.0, 66.4)
- added U8: CXP0650-220M-AG(22UH), easyeda2kicad:IND-SMD_L7.1-W6.6_CXP0650, F.Cu at (67.8, 73.9)
- added U9: TPS25740ARGER, easyeda2kicad:VQFN-24_L4.0-W4.0-P0.50-TL-EP, F.Cu at (88.1, 53.0)
- C11, C13, C23, C6: footprint Capacitor_SMD:CP_Elec_6.3x7.7 -> Capacitor_SMD:CP_Elec_8x10
- C18: renamed from C25; value 2u2 -> 22u
- C21: renamed from C17; footprint Capacitor_SMD:CP_Elec_6.3x7.7 -> Capacitor_SMD:CP_Elec_8x10
- C22, C26: value 2u2 -> 22u
- C22: renamed from C12; footprint Capacitor_SMD:CP_Elec_6.3x7.7 -> Capacitor_SMD:CP_Elec_8x10
- C4: renamed from C5; footprint Capacitor_SMD:CP_Elec_6.3x7.7 -> Capacitor_SMD:CP_Elec_8x10
- C5: renamed from C7; footprint Capacitor_SMD:CP_Elec_6.3x7.7 -> Capacitor_SMD:CP_Elec_8x10
- C8: value 100n -> 22u; footprint Capacitor_SMD:C_0603_1608Metric -> easyeda2kicad:C1812
- R21: value 4K02 -> 100K
- R22: value 100K -> 8K
- R28, R29: value 4K02 -> 10K
- R38: renamed from R5; value 20R -> 22R
- R39: value 4K02 -> 18K
- R4, R6: value 20R -> 22R
- R42: value 100K -> 10K
- R6: renamed from R14; value 20R -> 22R
- moved R28 85.4 mm to (83.3, 51.3)
- moved R29 84.9 mm to (83.3, 53.3)
- moved R31 84.0 mm to (83.3, 55.3)
- moved C14 82.5 mm to (76.9, 59.1), turned to 0 degrees
- moved R22 75.8 mm to (80.3, 53.3), turned to 0 degrees
- moved R21 75.8 mm to (80.3, 51.3)
- moved C8 71.4 mm to (82.7, 73.0), turned to 0 degrees
- moved R42 53.1 mm to (94.3, 86.8)
- moved R39 52.0 mm to (94.3, 82.8), turned to 0 degrees
- renumbered C15 to C19, C3 to C2, C10 to C20, C4 to C3, C18 to C6, C19 to C7, D13 to D4, J3 to J1, J4 to J2, J5 to J3, R34 to R10, R13 to R11, R35 to R12, R7 to R13, R8 to R14, R9 to R15, R10 to R16, R11 to R17, R12 to R18, R41 to R19, R40 to R20, R25 to R34, R26 to R35, R27 to R36, R3 to R4, R23 to R40, R2 to R5, R1 to R7, R20 to R8, R30 to R9, U4 to U10, U13 to U11, U9 to U2, U10 to U3, U11 to U4, U8 to U5, U15 to U6
Connections:
- C14 pad 1: Net-(C14-Pad1) -> Net-(U9-VAUX)
- C8 pad 1: Net-(C8-Pad1) -> GND
- C8 pad 2: GND -> +24V
- J1 pad 1: /USB_PD/USB2_VBUS -> +5V
- J1 pad 10: /USB_PD/USB2_GND -> GND
- J1 pad 4: /USB_PD/USB2_GND -> GND
- J1 pad 7: /USB_PD/USB2_GND -> GND
- J2 pad 1: /USB_PD1/USB2_VBUS -> +5V
- J2 pad 10: /USB_PD1/USB2_GND -> GND
- J2 pad 4: /USB_PD1/USB2_GND -> GND
- J2 pad 7: /USB_PD1/USB2_GND -> GND
- J3 pad 1: /USB_PD2/USB2_VBUS -> +5V
- J3 pad 10: /USB_PD2/USB2_GND -> GND
- J3 pad 4: /USB_PD2/USB2_GND -> GND
- J3 pad 7: /USB_PD2/USB2_GND -> GND
- R21 pad 1: Net-(C8-Pad1) -> Net-(U7-CSN2)
- R21 pad 2: Net-(U3-OPTO) -> Net-(R21-Pad2)
- R22 pad 1: Net-(U3-OPTO) -> Net-(U7-FB)
- R22 pad 2: Net-(U2-CSN2) -> Net-(R21-Pad2)
- R28 pad 1: Net-(C14-Pad1) -> Net-(Q1-G1)
- R28 pad 2: Net-(U5-VFB) -> Net-(U9-GDNG)
- R29 pad 1: Net-(C14-Pad1) -> Net-(U9-GDNG)
- R29 pad 2: Net-(U5-OPTO) -> Net-(C13-Pad1)
- R31 pad 1: Net-(U5-OPTO) -> Net-(U9-VAUX)
- R31 pad 2: Net-(U4-CSN2) -> Net-(U9-PCTRL)
- R34 pad 1: Net-(U4-CSN2) -> Net-(U10-CSN2)
- R34 pad 2: Net-(U5-VFB) -> Net-(R34-Pad2)
- R35 pad 1: Net-(U4-FB) -> Net-(U10-FB)
- R35 pad 2: Net-(U5-VFB) -> Net-(R34-Pad2)
- R36 pad 1: Net-(U4-FB) -> Net-(U10-FB)
- R39 pad 1: Net-(C20-Pad1) (its old number) -> Net-(U10-FB)
- R39 pad 2: Net-(U7-OPTO) -> /USB_PD3/CTL1
- R40 pad 2: Net-(U4-CSN2) -> Net-(U10-CSN2)
- R42 pad 1: Net-(U7-OPTO) -> Net-(U12-GDNG)
- R42 pad 2: Net-(U6-CSN2) -> Net-(C23-Pad1)
- U10 pad 1: Net-(U4-FB) -> Net-(U10-FB)
- U10 pad 4: Net-(U4-CSN2) -> Net-(U10-CSN2)
- U2 pad 2: /A_SSRX+ -> /A_SSTX+
- U2 pad 3: /A_SSRX- -> /A_SSTX-
- U2 pad 6: /A_SSTX+ -> /A_SSRX+
- U2 pad 7: /A_SSTX- -> /A_SSRX-
- U3 pad 2: /B_SSRX+ -> /B_SSTX+
- U3 pad 3: /B_SSRX- -> /B_SSTX-
- U3 pad 6: /B_SSTX+ -> /B_SSRX+
- U3 pad 7: /B_SSTX- -> /B_SSRX-
- U3 pad 10: /A_D- -> unconnected-(U3-DM2-Pad10)
- U3 pad 3: Net-(U3-OPTO) -> unconnected-(U3-OPTO-Pad3)
- U3 pad 9: /A_D+ -> unconnected-(U3-DP2-Pad9)
- U4 pad 2: /C_SSRX+ -> /C_SSTX+
- U4 pad 3: /C_SSRX- -> /C_SSTX-
- U4 pad 6: /C_SSTX+ -> /C_SSRX+
- U4 pad 7: /C_SSTX- -> /C_SSRX-
- U5 pad 10: /C_D- -> unconnected-(U5-DM2-Pad10)
- U5 pad 3: Net-(U5-OPTO) -> unconnected-(U5-OPTO-Pad3)
- U5 pad 9: /C_D+ -> unconnected-(U5-DP2-Pad9)
- U7 pad 10: /B_D- -> unconnected-(U7-DM2-Pad10)
- U7 pad 3: Net-(U7-OPTO) -> unconnected-(U7-OPTO-Pad3)
- U7 pad 9: /B_D+ -> unconnected-(U7-DP2-Pad9)
Routing:
- net /A_D-: track 44.5 -> 9.53 mm, vias 2 -> 1
- net /A_D+: track 46.1 -> 11.3 mm, vias 3 -> 2
- net unconnected-(U5-OPTO-Pad3): track 0.00 -> 25.0 mm, vias 0 -> 2
- net Net-(U5-OPTO): track 25.0 -> 0.00 mm, vias 2 -> 0
- net Net-(U3-OPTO): track 19.2 -> 0.00 mm, vias 2 -> 0
- net Net-(U4-FB): track 17.4 -> 0.00 mm, vias 2 -> 0
- net Net-(U10-FB): track 0.00 -> 17.4 mm, vias 0 -> 2
- net GND: track 162.4 -> 179.0 mm, vias 61 -> 67
- net unconnected-(U7-OPTO-Pad3): track 0.00 -> 15.8 mm, vias 0 -> 2
- net Net-(U7-OPTO): track 15.8 -> 0.00 mm, vias 2 -> 0
- net /C_SSRX-: track 50.1 -> 35.4 mm
- net Net-(U2-SEL): track 12.7 -> 0.00 mm
- net /C_SSTX-: track 34.8 -> 47.3 mm
- net /C_SSRX+: track 47.4 -> 35.1 mm
- net /C_SSTX+: track 34.8 -> 45.0 mm
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