File: USB_PD_Twitch/USB_PD_Twitch.kicad_sch (KiCad schematic)
At the start: 38 parts, among them J3 USB3_A, J4 USB3_A, J5 USB3_A, U1 NDP1360KC, U10 CH482D, U11 CH482D, U15 LM317L_SOT-89, U8 CXP0650-220M-AG(22UH), U9 CH482D

Commit message: add nev versions. (usb c and displayport working)
Parts:
- C5, C7: footprint Capacitor_SMD:CP_Elec_6.3x7.7 -> Capacitor_SMD:CP_Elec_8x10
Connections:
- net A_D+: no longer R8.2
- net A_D-: no longer R7.1
- net A_SSRX+: now also U9.6 (SSBX); no longer U9.2 (SSAX)
- net A_SSRX-: now also U9.7 (SSBY); no longer U9.3 (SSAY)
- net A_SSTX+: now also U9.2 (SSAX); no longer U9.6 (SSBX)
- net A_SSTX-: now also U9.3 (SSAY); no longer U9.7 (SSBY)
- net B_D+: no longer R10.2
- net B_D-: no longer R9.1
- net B_SSRX+: now also U10.6 (SSBX); no longer U10.2 (SSAX)
- net B_SSRX-: now also U10.7 (SSBY); no longer U10.3 (SSAY)
- net B_SSTX+: now also U10.2 (SSAX); no longer U10.6 (SSBX)
- net B_SSTX-: now also U10.3 (SSAY); no longer U10.7 (SSBY)
- net C_D+: no longer R12.2
- net C_D-: no longer R11.1
- net C_SSRX+: now also U11.6 (SSBX); no longer U11.2 (SSAX)
- net C_SSRX-: now also U11.7 (SSBY); no longer U11.3 (SSAY)
- net C_SSTX+: now also U11.2 (SSAX); no longer U11.6 (SSBX)
- net C_SSTX-: now also U11.3 (SSAY); no longer U11.7 (SSBY)
- new net USB_PD/USB2_D+: R8.2
- new net USB_PD/USB2_D-: R7.1
- new net USB_PD1/USB2_D+: R10.2
- new net USB_PD1/USB2_D-: R9.1
- new net USB_PD2/USB2_D+: R12.2
- new net USB_PD2/USB2_D-: R11.1
