File: USB_PD_PLUS_C/untitled.kicad_sch (KiCad schematic)
At the start: 28 parts, among them Q2 FS8205A_C908265, U10 NDP1360KC, U11 CXP0650-220M-AG(22UH), U12 TPS25740ARGER

Commit message: Update Schematic to 3 Port USB-C Power
I updated the schamtic to 3 port usb-C with superspeed and PD working
Parts:
- renumbered C28 to C29, C18 to C30, C19 to C31, C20 to C32, C21 to C33, C22 to C34, C23 to C35, C24 to C36, C25 to C37, C26 to C38, C27 to C39, Q2 to Q3, R34 to R47, R35 to R48, R36 to R49, R37 to R50, R38 to R51, R39 to R52, R40 to R53, R41 to R54, R42 to R55, R43 to R56, R44 to R57, R45 to R58, R46 to R59, U10 to U13, U11 to U14, U12 to U15

Commit message: update USB PD PCB to 3 in 3 out
Parts:
- removed C33, C34: 100u, Capacitor_SMD:CP_Elec_8x10, symbol Device:C_Polarized
- added C10, C11: 22u, easyeda2kicad:C1812, symbol Device:C
Connections:
- net GND: now also C10.2, C11.2
- net at C29.1, R53.1, U13.2 (CSP)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: now also C10.1, C11.1

Commit message: update routing usb c pd
Parts:
- removed R48: 8K, Resistor_SMD:R_0402_1005Metric, symbol Device:R
- C29, C31, C32, C35, C36, C37, C38, C39: footprint Capacitor_SMD:C_0603_1608Metric -> Capacitor_SMD:C_0402_1005Metric; LCSC C5137636 -> C5142567
- R47: value 100K -> 107K; LCSC C3017514 -> C25743
Connections:
- net at R49.1, R50.1, R52.1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: now also R47.2
Changed lines of the file:
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@@
 	(wire
 		(pts
+			(xy 40.64 83.82) (xy 40.64 91.44)
+		)
+		(stroke
+			(width 0)
+			(type default)
+		)
+	)
+	(wire
+		(pts
 			(xy 265.43 69.85) (xy 267.97 69.85)
 		)
@@
 			)
 		)
-		(property "Footprint" "Capacitor_SMD:C_0603_1608Metric"
+		(property "Footprint" "Capacitor_SMD:C_0402_1005Metric"
 			(at 238.4552 113.03 0)
 			(hide yes)
@@
 			)
 		)
-		(property "LCSC" "C5137636"
+		(property "LCSC" "C5142567"
 			(at 237.49 109.22 0)
 			(hide yes)
@@
 			)
 		)
-		(property "Footprint" "Capacitor_SMD:C_0603_1608Metric"
+		(property "Footprint" "Capacitor_SMD:C_0402_1005Metric"
 			(at 73.66 61.2648 0)
 			(hide yes)
@@
 			)
 		)
-		(property "LCSC" "C5137636"
+		(property "LCSC" "C5142567"
 			(at 69.85 62.23 90)
 			(hide yes)
@@
 			)
 		)
-		(property "Footprint" "Capacitor_SMD:C_0603_1608Metric"
+		(property "Footprint" "Capacitor_SMD:C_0402_1005Metric"
 			(at 16.2052 69.85 0)
 			(hide yes)
@@
 			)
 		)
-		(property "LCSC" "C5137636"
+		(property "LCSC" "C5142567"
 			(at 15.24 66.04 0)
 			(hide yes)
@@
 			)
 		)
-		(property "Footprint" "Capacitor_SMD:C_0603_1608Metric"
+		(property "Footprint" "Capacitor_SMD:C_0402_1005Metric"
 			(at 129.2352 90.17 0)
 			(hide yes)
@@
 			)
 		)
-		(property "LCSC" "C5137636"
+		(property "LCSC" "C5142567"
 			(at 128.27 86.36 0)
 			(hide yes)
@@
 			)
 		)
-		(property "Value" "100K"
-			(at 40.64 82.804 90)
+		(property "Value" "107K"
+			(at 40.64 82.55 90)
 			(show_name no)
 			(do_not_autoplace no)
@@
 			)
 		)
-		(property "LCSC" "C3017514"
+		(property "LCSC" "C25743"
 			(at 40.64 80.01 0)
 			(hide yes)
@@
 			)
 		)
-		(property "Footprint" "Capacitor_SMD:C_0603_1608Metric"
+		(property "Footprint" "Capacitor_SMD:C_0402_1005Metric"
 			(at 176.8348 69.85 0)
 			(hide yes)
@@
 			)
 		)
-		(property "LCSC" "C5137636"
+		(property "LCSC" "C5142567"
 			(at 177.8 73.66 0)
 			(hide yes)
@@
 	(symbol
 		(lib_id "Device:R")
-		(at 40.64 87.63 180)
-		(unit 1)
-		(body_style 1)
-		(exclude_from_sim no)
-		(in_bom yes)
-		(on_board yes)
-		(in_pos_files yes)
-		(dnp no)
-		(property "Reference" "R48"
-			(at 39.624 86.614 0)
-			(show_name no)
-			(do_not_autoplace no)
-			(effects
-				(font
-					(size 1.27 1.27)
-				)
-				(justify left)
-			)
-		)
-		(property "Value" "8K"
-			(at 40.64 86.106 90)
-			(show_name no)
-			(do_not_autoplace no)
-			(effects
-				(font
-					(size 1.27 1.27)
-				)
-				(justify left)
-			)
-		)
-		(property "Footprint" "Resistor_SMD:R_0402_1005Metric"
-			(at 42.418 87.63 90)
-			(hide yes)
-			(show_name no)
-			(do_not_autoplace no)
-			(effects
-				(font
-					(size 1.27 1.27)
-				)
-			)
-		)
-		(property "Datasheet" ""
-			(at 40.64 87.63 0)
-			(hide yes)
-			(show_name no)
-			(do_not_autoplace no)
-			(effects
-				(font
-					(size 1.27 1.27)
-				)
-			)
-		)
-		(property "Description" "Resistor"
-			(at 40.64 87.63 0)
-			(hide yes)
-			(show_name no)
-			(do_not_autoplace no)
-			(effects
-				(font
-					(size 1.27 1.27)
-				)
-			)
-		)
-		(property "LCSC" "C2960789"
-			(at 40.64 87.63 0)
-			(hide yes)
-			(show_name no)
-			(do_not_autoplace no)
-			(effects
-				(font
-					(size 1.27 1.27)
-				)
-			)
-		)
-		(property "Sim.Device" ""
-			(at 40.64 87.63 0)
-			(hide yes)
-			(show_name no)
-			(do_not_autoplace no)
-			(effects
-				(font
-					(size 1.27 1.27)
-				)
-			)
-		)
-		(property "Sim.Type" ""
-			(at 40.64 87.63 0)
-			(hide yes)
-			(show_name no)
-			(do_not_autoplace no)
-			(effects
-				(font
-					(size 1.27 1.27)
-				)
-			)
-		)
-		(property "LCSC Part" "C2960789"
-			(at 40.64 87.63 0)
-			(hide yes)
-			(show_name no)
-			(do_not_autoplace no)
-			(effects
-				(font
-					(size 1.27 1.27)
-				)
-			)
-		)
-		(pin "1"
-		)
-		(pin "2"
-		)
-		(instances
-			(project "USB_PD_PLUS_C"
-				(path "/dc229072-24b4-43c8-b91f-e7db21590dc5/5dcbd05b-b508-4a41-bbc9-03ae250f4faf"
-					(reference "R35")
-					(unit 1)
-				)
-				(path "/dc229072-24b4-43c8-b91f-e7db21590dc5/78c12fed-0488-4a52-9624-e29b3b05d9b8"
-					(reference "R61")
-					(unit 1)
-				)
-				(path "/dc229072-24b4-43c8-b91f-e7db21590dc5/ce440652-8abb-43f9-90a6-4d0613a82a69"
-					(reference "R48")
-					(unit 1)
-				)
-			)
-		)
-	)
-	(symbol
-		(lib_id "Device:R")
 		(at 176.53 80.01 90)
 		(unit 1)
@@
 			)
 		)
-		(property "Footprint" "Capacitor_SMD:C_0603_1608Metric"
+		(property "Footprint" "Capacitor_SMD:C_0402_1005Metric"
 			(at 61.9252 59.69 0)
 			(hide yes)
@@
 			)
 		)
-		(property "LCSC" "C5137636"
+		(property "LCSC" "C5142567"
 			(at 60.96 55.88 0)
 			(hide yes)
@@
 			)
 		)
-		(property "Footprint" "Capacitor_SMD:C_0603_1608Metric"
+		(property "Footprint" "Capacitor_SMD:C_0402_1005Metric"
 			(at 167.9448 69.85 0)
 			(hide yes)
@@
 			)
 		)
-		(property "LCSC" "C5137636"
+		(property "LCSC" "C5142567"
 			(at 168.91 73.66 0)
 			(hide yes)
@@
 			)
 		)
-		(property "Footprint" "Capacitor_SMD:C_0603_1608Metric"
+		(property "Footprint" "Capacitor_SMD:C_0402_1005Metric"
 			(at 184.4548 69.85 0)
 			(hide yes)
@@
 			)
 		)
-		(property "LCSC" "C5137636"
+		(property "LCSC" "C5142567"
 			(at 185.42 73.66 0)
 			(hide yes)
